File: aquarium.sch (KiCad schematic (older format))
At the start: 0 parts

Commit message: create the electronics schema
Parts:
- added A1: Arduino Nano, Module:Arduino_Nano, symbol MCU_Module:Arduino_Nano_v3.x
- added C1, C3: 1u-100u, symbol Device:C
- added C2: 0.1u-1u, symbol Device:C
- added J1: DC Input, symbol Connector:Barrel_Jack
- added J2: LED 1 Output, symbol Connector:Barrel_Jack
- added J3: LED 2 Output, symbol Connector:Barrel_Jack
- added Q1: IRLZ44N, Package_TO_SOT_THT:TO-220-3_Vertical, symbol Transistor_FET:IRLZ44N
- added R1, R2: 100k, symbol Device:R
- added RV1: Gradient time, symbol Device:R_POT
- added SW1: Interval reset, symbol Switch:SW_Push
- added SW2: Power switch, symbol Switch:SW_SPDT
- added U1: DS3231, Package_SO:SOIC-16W_7.5x10.3mm_P1.27mm, symbol Timer_RTC:DS3231M
- added U2: TC4426ACPA, symbol symbols:TC4426ACPA
Connections:
- new net: Q1.1 (G), U2.7 (Output_A)
- new net +12V: A1.30 (VIN), C1.1, C3.1, J2.1, J3.1, SW2.1 (A), U2.6 (VDD)
- new net +5V: A1.27 (+5V), C2.1, R1.1, R2.1, RV1.1, U1.2 (VCC)
- new net GND: A1.29 (GND), A1.4 (GND), C1.2, C2.2, C3.2, J1.2, Q1.3 (S), RV1.3, SW1.1, U1.10 (GND), U1.11 (GND), U1.12 (GND), U1.13 (GND), U1.5 (GND), U1.6 (GND), U1.7 (GND), U1.8 (GND), U1.9 (GND), U2.3 (GND)
- new net INT: A1.5 (D2), R2.2, U1.3 (~INT~/SQW)
- new net IN_GRAD: A1.21 (A2), RV1.2
- new net IN_RESET: A1.6 (D3), R1.2, SW1.2
- new net MOSFET: A1.14 (D11), U2.2 (Input_A)
- new net OUT_LED: J2.2, J3.2, Q1.2 (D)
- new net SCL: A1.24 (A5), U1.16 (SCL)
- new net SDA: A1.23 (A4), U1.15 (SDA)
- new net VCC_CON: J1.1, SW2.2 (B)
- no-connect marks 0 -> 26
Other:
- note added: "Arduino"
- note added: "Connectors and inputs"
- note added: "MOSFET"
- note added: "RTC"

Commit message: add an error led
Parts:
- added D?: RED, symbol Device:LED
- added R?: 1k, symbol Device:R
Connections:
- net GND: now also D?.1 (K)
- net LED_ERROR: now reaches A1.7 (D4)
- net LED_ERROR: now also R?.1
- new net: D?.2 (A), R?.2
- no-connect marks 26 -> 25
Changed lines of the file:
@@
 Text GLabel 2150 1450 0    50   Input ~ 0
 SDA
-Text GLabel 3150 1650 2    50   Input ~ 0
-INT
 Text GLabel 3900 1650 3    50   Input ~ 0
 INT
@@
 Text GLabel 4100 5750 2    50   Input ~ 0
 SDA
-Text GLabel 3100 4950 0    50   Input ~ 0
-INT
 Text GLabel 4100 5550 2    50   Input ~ 0
 IN_GRAD
@@
 NoConn ~ 3100 5350
 NoConn ~ 3100 5250
-NoConn ~ 3100 5150
 NoConn ~ 3100 4850
 NoConn ~ 3100 4750
+Text GLabel 3100 5150 0    50   Input ~ 0
+LED_ERROR
+Text GLabel 3100 4950 0    50   Input ~ 0
+INT
+Text GLabel 3150 1650 2    50   Input ~ 0
+INT
+$Comp
+L Device:R R?
+U 1 1 5F8DB3E4
+P 5500 3750
+F 0 "R?" H 5600 3850 50  0000 L CNN
+F 1 "1k" H 5600 3650 50  0000 L CNN
+F 2 "" V 5430 3750 50  0001 C CNN
+F 3 "~" H 5500 3750 50  0001 C CNN
+	1    5500 3750
+	1    0    0    -1
+$EndComp
+$Comp
+L Device:LED D?
+U 1 1 5F8DC9F3
+P 5500 4150
+F 0 "D?" V 5600 4050 50  0000 R CNN
+F 1 "RED" V 5350 4050 50  0000 R CNN
+F 2 "" H 5500 4150 50  0001 C CNN
+F 3 "~" H 5500 4150 50  0001 C CNN
+	1    5500 4150
+	0    -1   -1   0
+$EndComp
+Wire Wire Line
+	5500 4000 5500 3900
+$Comp
+L power:GND #PWR?
+U 1 1 5F8DDDCC
+P 5500 4400
+F 0 "#PWR?" H 5500 4150 50  0001 C CNN
+F 1 "GND" H 5500 4250 50  0000 C CNN
+F 2 "" H 5500 4400 50  0001 C CNN
+F 3 "" H 5500 4400 50  0001 C CNN
+	1    5500 4400
+	1    0    0    -1
+$EndComp
+Wire Wire Line
+	5500 4400 5500 4300
+Text GLabel 5500 3550 1    50   Input ~ 0
+LED_ERROR
+Wire Wire Line
+	5500 3550 5500 3600
 $EndSCHEMATC

Commit message: remove the external pullup resistor for the interrupt pin
Parts:
- removed R2: 100k, symbol Device:R
Other:
- note added: "Use INPUT_PULLUP in Arduino for D2"
Changed lines of the file:
@@
 Title "Aquarium clock-driven LED dimmer"
 Date "2020-10-07"
-Rev "v1.0"
+Rev "v1.1"
 Comp "Martin Jakubik"
 Comment1 ""
@@
 Text GLabel 2150 1450 0    50   Input ~ 0
 SDA
-Text GLabel 3900 1650 3    50   Input ~ 0
-INT
-$Comp
-L Device:R R2
-U 1 1 5F826462
-P 3900 1450
-F 0 "R2" H 4000 1550 50  0000 L CNN
-F 1 "100k" H 4000 1350 50  0000 L CNN
-F 2 "" V 3830 1450 50  0001 C CNN
-F 3 "~" H 3900 1450 50  0001 C CNN
-	1    3900 1450
-	1    0    0    -1
-$EndComp
-Wire Wire Line
-	3900 1600 3900 1650
-$Comp
-L power:+5V #PWR05
-U 1 1 5F826E2F
-P 3900 1250
-F 0 "#PWR05" H 3900 1100 50  0001 C CNN
-F 1 "+5V" H 3900 1400 50  0000 C CNN
-F 2 "" H 3900 1250 50  0001 C CNN
-F 3 "" H 3900 1250 50  0001 C CNN
-	1    3900 1250
-	1    0    0    -1
-$EndComp
-Wire Wire Line
-	3900 1250 3900 1300
 Wire Notes Line
 	470  2700 11220 2700
@@
 Wire Wire Line
 	5500 3550 5500 3600
+Text Notes 2900 4900 2    50   ~ 0
+Use INPUT_PULLUP in Arduino for D2
 $EndSCHEMATC

Commit message: assign footprints
Parts:
- C1, C2, C3: footprint (none) -> Capacitor_THT:C_Disc_D5.0mm_W2.5mm_P2.50mm
- D1: renamed from D?; footprint (none) -> LED_THT:LED_D5.0mm
- J1, J2, J3: footprint (none) -> Connector_BarrelJack:BarrelJack_Horizontal
- R1: footprint (none) -> Resistor_THT:R_Axial_DIN0207_L6.3mm_D2.5mm_P10.16mm_Horizontal
- R2: renamed from R?; footprint (none) -> Resistor_THT:R_Axial_DIN0207_L6.3mm_D2.5mm_P10.16mm_Horizontal
- RV1, SW2: footprint (none) -> Connector_JST:JST_XH_B3B-XH-A_1x03_P2.50mm_Vertical
- SW1: footprint (none) -> Connector_JST:JST_XH_B2B-XH-A_1x02_P2.50mm_Vertical
- U1: footprint Package_SO:SOIC-16W_7.5x10.3mm_P1.27mm -> Connector_JST:JST_XH_B6B-XH-A_1x06_P2.50mm_Vertical
- U2: footprint (none) -> Package_DIP:DIP-8_W7.62mm_Socket
Changed lines of the file:
@@
 F 0 "U1" H 3000 1900 50  0000 C CNN
 F 1 "DS3231" H 2900 1200 50  0000 C CNN
-F 2 "Package_SO:SOIC-16W_7.5x10.3mm_P1.27mm" H 2650 950 50  0001 C CNN
+F 2 "Connector_JST:JST_XH_B6B-XH-A_1x06_P2.50mm_Vertical" H 2650 950 50  0001 C CNN
 F 3 "http://datasheets.maximintegrated.com/en/ds/DS3231.pdf" H 2920 1600 50  0001 C CNN
 	1    2650 1550
@@
 F 0 "J1" H 5450 1400 50  0000 C CNN
 F 1 "DC Input" H 5450 1000 50  0000 C CNN
-F 2 "" H 5500 1160 50  0001 C CNN
+F 2 "Connector_BarrelJack:BarrelJack_Horizontal" H 5500 1160 50  0001 C CNN
 F 3 "~" H 5500 1160 50  0001 C CNN
 	1    5450 1200
@@
 F 0 "U2" H 9500 5200 50  0000 C CNN
 F 1 "TC4426ACPA" H 9550 4200 50  0000 C CNN
-F 2 "" H 9250 4700 50  0001 C CNN
+F 2 "Package_DIP:DIP-8_W7.62mm_Socket" H 9250 4700 50  0001 C CNN
 F 3 "https://www.distrelec.sk/Web/Downloads/_t/ds/TC4426A_24A_28Ax_eng_tds.pdf" H 9250 4700 50  0001 C CNN
 	1    9250 4700
@@
 F 0 "SW2" H 5850 2300 50  0000 C CNN
 F 1 "Power switch" H 5850 1900 50  0000 C CNN
-F 2 "" H 5850 2100 50  0001 C CNN
+F 2 "Connector_JST:JST_XH_B3B-XH-A_1x03_P2.50mm_Vertical" H 5850 2100 50  0001 C CNN
 F 3 "~" H 5850 2100 50  0001 C CNN
 	1    5850 2100
@@
 F 0 "SW1" H 8600 1300 50  0000 C CNN
 F 1 "Interval reset" H 8600 1000 50  0000 C CNN
-F 2 "" H 8600 1300 50  0001 C CNN
+F 2 "Connector_JST:JST_XH_B2B-XH-A_1x02_P2.50mm_Vertical" H 8600 1300 50  0001 C CNN
 F 3 "~" H 8600 1300 50  0001 C CNN
 	1    8600 1100
@@
 F 0 "RV1" H 7150 1750 50  0000 R CNN
 F 1 "Gradient time" H 7150 1550 50  0000 R CNN
-F 2 "" H 7250 1650 50  0001 C CNN
+F 2 "Connector_JST:JST_XH_B3B-XH-A_1x03_P2.50mm_Vertical" H 7250 1650 50  0001 C CNN
 F 3 "~" H 7250 1650 50  0001 C CNN
 	1    7250 1650
@@
 F 0 "J2" H 10150 1500 50  0000 C CNN
 F 1 "LED 1 Output" H 10150 1100 50  0000 C CNN
-F 2 "" H 10200 1260 50  0001 C CNN
+F 2 "Connector_BarrelJack:BarrelJack_Horizontal" H 10200 1260 50  0001 C CNN
 F 3 "~" H 10200 1260 50  0001 C CNN
 	1    10150 1300
@@
 F 0 "J3" H 10150 2300 50  0000 C CNN
 F 1 "LED 2 Output" H 10150 1900 50  0000 C CNN
-F 2 "" H 10200 2060 50  0001 C CNN
+F 2 "Connector_BarrelJack:BarrelJack_Horizontal" H 10200 2060 50  0001 C CNN
 F 3 "~" H 10200 2060 50  0001 C CNN
 	1    10150 2100
@@
 F 0 "C1" H 1800 3700 50  0000 L CNN
 F 1 "1u-100u" H 1800 3600 50  0000 L CNN
-F 2 "" H 1738 3500 50  0001 C CNN
+F 2 "Capacitor_THT:C_Disc_D5.0mm_W2.5mm_P2.50mm" H 1738 3500 50  0001 C CNN
 F 3 "~" H 1700 3650 50  0001 C CNN
 	1    1700 3650
@@
 F 0 "R1" H 8750 1950 50  0000 L CNN
 F 1 "100k" H 8750 1750 50  0000 L CNN
-F 2 "" V 8580 1850 50  0001 C CNN
+F 2 "Resistor_THT:R_Axial_DIN0207_L6.3mm_D2.5mm_P10.16mm_Horizontal" V 8580 1850 50  0001 C CNN
 F 3 "~" H 8650 1850 50  0001 C CNN
 	1    8650 1850
@@
 F 0 "C2" H 1350 1500 50  0000 L CNN
 F 1 "0.1u-1u" H 1350 1400 50  0000 L CNN
-F 2 "" H 1288 1300 50  0001 C CNN
+F 2 "Capacitor_THT:C_Disc_D5.0mm_W2.5mm_P2.50mm" H 1288 1300 50  0001 C CNN
 F 3 "~" H 1250 1450 50  0001 C CNN
 	1    1250 1450
@@
 F 0 "C3" H 7700 4650 50  0000 L CNN
 F 1 "1u-100u" H 7700 4550 50  0000 L CNN
-F 2 "" H 7638 4450 50  0001 C CNN
+F 2 "Capacitor_THT:C_Disc_D5.0mm_W2.5mm_P2.50mm" H 7638 4450 50  0001 C CNN
 F 3 "~" H 7600 4600 50  0001 C CNN
 	1    7600 4600
@@
 INT
 $Comp
-L Device:R R?
+L Device:R R2
 U 1 1 5F8DB3E4
 P 5500 3750
-F 0 "R?" H 5600 3850 50  0000 L CNN
+F 0 "R2" H 5600 3850 50  0000 L CNN
 F 1 "1k" H 5600 3650 50  0000 L CNN
-F 2 "" V 5430 3750 50  0001 C CNN
+F 2 "Resistor_THT:R_Axial_DIN0207_L6.3mm_D2.5mm_P10.16mm_Horizontal" V 5430 3750 50  0001 C CNN
 F 3 "~" H 5500 3750 50  0001 C CNN
 	1    5500 3750
@@
 $EndComp
 $Comp
-L Device:LED D?
+L Device:LED D1
 U 1 1 5F8DC9F3
 P 5500 4150
-F 0 "D?" V 5600 4050 50  0000 R CNN
+F 0 "D1" V 5600 4050 50  0000 R CNN
 F 1 "RED" V 5350 4050 50  0000 R CNN
-F 2 "" H 5500 4150 50  0001 C CNN
+F 2 "LED_THT:LED_D5.0mm" H 5500 4150 50  0001 C CNN
 F 3 "~" H 5500 4150 50  0001 C CNN
 	1    5500 4150
@@
 	5500 4000 5500 3900
 $Comp
-L power:GND #PWR?
+L power:GND #PWR05
 U 1 1 5F8DDDCC
 P 5500 4400
-F 0 "#PWR?" H 5500 4150 50  0001 C CNN
+F 0 "#PWR05" H 5500 4150 50  0001 C CNN
 F 1 "GND" H 5500 4250 50  0000 C CNN
 F 2 "" H 5500 4400 50  0001 C CNN

Commit message: create a simple pcb design
This is an inspiration for the proofboard
design I'm going to solder.
Parts:
- J1: Comment (none) -> 12V, max 1.5A
Changed lines of the file:
@@
 F 2 "Connector_BarrelJack:BarrelJack_Horizontal" H 5500 1160 50  0001 C CNN
 F 3 "~" H 5500 1160 50  0001 C CNN
+F 4 "12V, max 1.5A" H 5450 900 50  0000 C CIN "Comment"
 	1    5450 1200
 	1    0    0    -1
@@
 L power:GND #PWR06
 U 1 1 5F7E8F3A
-P 5800 1350
-F 0 "#PWR06" H 5800 1100 50  0001 C CNN
-F 1 "GND" H 5800 1200 50  0000 C CNN
-F 2 "" H 5800 1350 50  0001 C CNN
-F 3 "" H 5800 1350 50  0001 C CNN
-	1    5800 1350
-	1    0    0    -1
-$EndComp
-Wire Wire Line
-	5800 1350 5800 1300
-Wire Wire Line
-	5800 1300 5750 1300
+P 6100 1350
+F 0 "#PWR06" H 6100 1100 50  0001 C CNN
+F 1 "GND" H 6100 1200 50  0000 C CNN
+F 2 "" H 6100 1350 50  0001 C CNN
+F 3 "" H 6100 1350 50  0001 C CNN
+	1    6100 1350
+	1    0    0    -1
+$EndComp
 $Comp
 L Device:C C1
@@
 Text Notes 2900 4900 2    50   ~ 0
 Use INPUT_PULLUP in Arduino for D2
+Wire Wire Line
+	6100 1350 6100 1300
+Wire Wire Line
+	5750 1300 6100 1300
 $EndSCHEMATC

Commit message: update the schematic to the actual parts used for soldering
Parts:
- removed SW2: Power switch, Connector_JST:JST_XH_B3B-XH-A_1x03_P2.50mm_Vertical, symbol Switch:SW_SPDT
- removed U1: DS3231, Connector_JST:JST_XH_B6B-XH-A_1x06_P2.50mm_Vertical, symbol Timer_RTC:DS3231M
- removed U2: TC4426ACPA, Package_DIP:DIP-8_W7.62mm_Socket, symbol symbols:TC4426ACPA
- added C3: 0.1u, Capacitor_THT:C_Disc_D5.0mm_W2.5mm_P2.50mm, symbol Device:C
- added U1: DS3231, Connector_PinHeader_2.54mm:PinHeader_1x06_P2.54mm_Vertical, symbol symbols:DS3231
- added U2: MIC4420BN, Package_DIP:DIP-8_W7.62mm_Socket, symbol symbols:MIC4420BN
- C1: value 1u-100u -> 10u
- C2: value 0.1u-1u -> 0.1u
- C4: renamed from C3; value 1u-100u -> 10u
Connections:
- net VCC_CON is gone; now on net +12V: J1.1
- net +12V: now also U2.1 (VCC), U2.8 (VCC)
- net +5V: now also C3.1, U1.5 (VCC)
- net GND: now also C3.2, U1.6 (GND), U2.4 (GND), U2.5 (GND)
- net INT: now also U1.2 (SQW)
- net MOSFET: now also U2.2 (IN)
- net SCL: now also U1.3 (SCL)
- net SDA: now also U1.4 (SDA)
- net MOSFET_OUT: now reaches Q1.1 (G)
- net MOSFET_OUT: now also U2.6 (OUT), U2.7 (OUT)
- no-connect marks 25 -> 20
Other:
- moved on the sheet: C2, R1, SW1
